File: rucheb.kicad_sch (KiCad schematic)
At the start: 23 parts, among them IC1 CN3791, J1 Conn_01x02, Q1 AO3401A

Commit message: update
Parts:
- added U7: 1043, Empreintes:1043, symbol 1043:1043
Connections:
- net GND: now also U7.2 (-)
- net VBAT: now also U7.1 (+)
Changed lines of the file:
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@@
+    (stroke (width 0) (type default) (color 0 0 0 0))
+  )
+  (wire (pts (xy 232.41 83.82) (xy 232.41 87.63))
     (stroke (width 0) (type default) (color 0 0 0 0))
   )
@@
     (stroke (width 0) (type default) (color 0 0 0 0))
   )
+  (wire (pts (xy 243.84 83.82) (xy 232.41 83.82))
+    (stroke (width 0) (type default) (color 0 0 0 0))
+  )
   (wire (pts (xy 116.84 41.91) (xy 116.84 46.99))
+    (stroke (width 0) (type default) (color 0 0 0 0))
+  )
+  (wire (pts (xy 238.76 81.28) (xy 243.84 81.28))
     (stroke (width 0) (type default) (color 0 0 0 0))
   )
@@
     (property "Intersheet References" "${INTERSHEET_REFS}" (id 0) (at 110.4106 27.3696 90)
       (effects (font (size 1.27 1.27)) (justify left) hide)
+    )
+  )
+  (global_label "VBAT" (shape input) (at 238.76 81.28 180) (fields_autoplaced)
+    (effects (font (size 1.27 1.27)) (justify right))
+    (property "Intersheet References" "${INTERSHEET_REFS}" (id 0) (at 232.021 81.2006 0)
+      (effects (font (size 1.27 1.27)) (justify right) hide)
     )
   )
@@
     (pin "1")
   )
+  (symbol (lib_id "power:GND") (at 232.41 87.63 0) (unit 1)
+    (in_bom yes) (on_board yes)
+    (property "Reference" "#PWR0103" (id 0) (at 232.41 93.98 0)
+      (effects (font (size 1.27 1.27)) hide)
+    )
+    (property "Value" "GND" (id 1) (at 232.537 92.0242 0))
+    (property "Footprint" "" (id 2) (at 232.41 87.63 0)
+      (effects (font (size 1.27 1.27)) hide)
+    )
+    (property "Datasheet" "" (id 3) (at 232.41 87.63 0)
+      (effects (font (size 1.27 1.27)) hide)
+    )
+    (pin "1")
+  )
   (symbol (lib_id "ruche-rescue:CP-Device") (at 227.33 50.8 0) (unit 1)
     (in_bom yes) (on_board yes)
@@
     (pin "1")
   )
+  (symbol (lib_id "1043:1043") (at 243.84 81.28 0) (unit 1)
+    (in_bom yes) (on_board yes) (fields_autoplaced)
+    (property "Reference" "U7" (id 0) (at 256.54 75.091 0))
+    (property "Value" "1043" (id 1) (at 256.54 77.6279 0))
+    (property "Footprint" "Empreintes:1043" (id 2) (at 265.43 78.74 0)
+      (effects (font (size 1.27 1.27)) (justify left) hide)
+    )
+    (property "Datasheet" "http://www.keyelco.com/product-pdf.cfm?p=919" (id 3) (at 265.43 81.28 0)
+      (effects (font (size 1.27 1.27)) (justify left) hide)
+    )
+    (property "Description" "KEYSTONE - 1043 - BATTERY HOLDER, 18650, TH" (id 4) (at 265.43 83.82 0)
+      (effects (font (size 1.27 1.27)) (justify left) hide)
+    )
+    (property "Height" "14.86" (id 5) (at 265.43 86.36 0)
+      (effects (font (size 1.27 1.27)) (justify left) hide)
+    )
+    (property "Mouser Part Number" "534-1043" (id 6) (at 265.43 88.9 0)
+      (effects (font (size 1.27 1.27)) (justify left) hide)
+    )
+    (property "Mouser Price/Stock" "https://www.mouser.co.uk/ProductDetail/Keystone-Electronics/1043?qs=%2F7TOpeL5Mz6j%2FnxeOA1rsg%3D%3D" (id 7) (at 265.43 91.44 0)
+      (effects (font (size 1.27 1.27)) (justify left) hide)
+    )
+    (property "Manufacturer_Name" "Keystone Electronics" (id 8) (at 265.43 93.98 0)
+      (effects (font (size 1.27 1.27)) (justify left) hide)
+    )
+    (property "Manufacturer_Part_Number" "1043" (id 9) (at 265.43 96.52 0)
+      (effects (font (size 1.27 1.27)) (justify left) hide)
+    )
+    (pin "1")
+    (pin "2")
+    (pin "MH1")
+    (pin "MH2")
+    (pin "MH3")
+  )
 )
