File: untitled.kicad_sch (KiCad schematic)
At the start: 60 parts, among them IC5 HX711, IC6 HX711, IC7 HX711, IC8 HX711, J10 Conn_01x05, J15 Conn_01x05, J16 Conn_01x05, J2 Conn_01x05, Q2 MMBT4403, Q3 MMBT4403, Q4 MMBT4403, Q5 MMBT4403

Commit message: update
Parts:
- removed J10, J15, J16, J2: Conn_01x05, Empreintes:connecteurs5, symbol Connector_Generic:Conn_01x05
- added J10, J15, J16, J2: Conn_01x04, Empreintes:1725672, symbol Connector_Generic:Conn_01x04
- added J6, J7: Conn_01x02, Empreintes:SHDR2W90P0X500_1X2_1060X980X1380P, symbol Connector_Generic:Conn_01x02
Connections:
- net GND: now also J10.3 (Pin_3), J15.3 (Pin_3), J16.3 (Pin_3), J2.3 (Pin_3), J6.1 (Pin_1), J6.2 (Pin_2), J7.1 (Pin_1), J7.2 (Pin_2)
- net at C37.1, C39.1, L5.1: now also J16.4 (Pin_4)
- net at C36.1, C38.1, L4.1: now also J15.4 (Pin_4)
- net at C23.1, C25.1, L3.1: now also J10.4 (Pin_4)
- net at R21.2: now also J10.2 (Pin_2)
- net at R22.2: now also J10.1 (Pin_1)
- net at C22.1, C24.1, L2.1: now also J2.4 (Pin_4)
- net at R29.2: now also J16.2 (Pin_2)
- net at R17.2: now also J2.2 (Pin_2)
- net at R18.2: now also J2.1 (Pin_1)
- net at R30.2: now also J16.1 (Pin_1)
- net at R25.2: now also J15.2 (Pin_2)
- net at R26.2: now also J15.1 (Pin_1)

Commit message: update
Connections:
- net CLK3: now also IC7.11 (PD_SCK); no longer IC8.11 (PD_SCK)
- net CLK4: now also IC8.11 (PD_SCK); no longer IC7.11 (PD_SCK)
- net DAT3: now also IC7.12 (DOUT); no longer IC8.12 (DOUT)
- net DAT4: now also IC8.12 (DOUT); no longer IC7.12 (DOUT)
Changed lines of the file:
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@@
     (stroke (width 0) (type default) (color 0 0 0 0))
   )
-  (global_label "CLK4" (shape output) (at 276.86 130.81 0) (fields_autoplaced)
+  (global_label "CLK3" (shape output) (at 276.86 130.81 0) (fields_autoplaced)
     (effects (font (size 1.27 1.27)) (justify left))
     (property "Intersheet References" "${INTERSHEET_REFS}" (id 0) (at 283.9618 130.7306 0)
@@
     )
   )
-  (global_label "CLK3" (shape output) (at 278.13 58.42 0) (fields_autoplaced)
+  (global_label "CLK4" (shape output) (at 278.13 58.42 0) (fields_autoplaced)
     (effects (font (size 1.27 1.27)) (justify left))
     (property "Intersheet References" "${INTERSHEET_REFS}" (id 0) (at 285.2318 58.3406 0)
@@
     )
   )
-  (global_label "DAT4" (shape output) (at 276.86 128.27 0) (fields_autoplaced)
+  (global_label "DAT3" (shape output) (at 276.86 128.27 0) (fields_autoplaced)
     (effects (font (size 1.27 1.27)) (justify left))
     (property "Intersheet References" "${INTERSHEET_REFS}" (id 0) (at 283.7199 128.1906 0)
@@
     )
   )
-  (global_label "DAT3" (shape output) (at 278.13 55.88 0) (fields_autoplaced)
+  (global_label "DAT4" (shape output) (at 278.13 55.88 0) (fields_autoplaced)
     (effects (font (size 1.27 1.27)) (justify left))
     (property "Intersheet References" "${INTERSHEET_REFS}" (id 0) (at 284.9899 55.8006 0)
