File: ruche.kicad_pcb (KiCad board)
At the start: 2 copper layers, 82.8 x 99.9 mm, 181 parts, among them IC1 CN3791, IC2 MAX17048G+, IC3 L86-M33, IC4 SHT41-AD1B-R3, IC5 HX711, IC6 HX711, IC7 HX711, IC8 HX711, J1 Conn_01x02, J10 Conn_01x05, J11 Conn_01x04, J12 Conn_01x04, J13 Micro_SD_Card, J14 Conn_01x03, J15 Conn_01x05, J16 Conn_01x05, J17 Conn_01x04, J18 Conn_01x04, J19 Conn_01x02, J2 Conn_01x05, J20 USB_C_Receptacle_USB2.0 USB41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, J3 Conn_01x03, J4 Conn_01x03, J5 Conn_01x04, J6 Conn_01x02, J7 Conn_01x02, J8 Conn_01x03, J9 Conn_01x03, Q1 AO3401A, Q2 MMBT4403, Q3 MMBT4403, Q4 MMBT4403, Q5 MMBT4403, Q6 UMH3N, Q7 DMG2301L, SW1 SW_Push, U1 CP2102N-A02-GQFN24, U2 MS5611-01BA, U3 XC6220B331MR, U4 TCA9548APWR, U5 XC6220B331MR, U6 ESP32-S3-WROOM-2

Commit message: update
Parts:
- removed D13: D_Schottky, Diode_SMD:D_SOD-323
- removed JP2: SolderJumper_2_Open, Jumper:SolderJumper-2_P1.3mm_Open_RoundedPad1.0x1.5mm
- added C60: 10µF, Capacitor_SMD:C_0603_1608Metric, F.Cu at (156.6, 156.4)
- added C61: 0.1µF, Capacitor_SMD:C_0805_2012Metric, F.Cu at (158.2, 156.5)
- added C62: 0.1µF, Capacitor_SMD:C_0603_1608Metric, F.Cu at (151.2, 156.4)
- added C63: 10µF, Capacitor_SMD:C_0805_2012Metric, F.Cu at (149.6, 156.5)
- added R50: 10K, Resistor_SMD:R_0603_1608Metric, F.Cu at (120.6, 109.3)
- added R51: 10K, Resistor_SMD:R_0603_1608Metric, F.Cu at (119.3, 109.3)
- added U7: 1043, Empreintes:1043, B.Cu at (168.1, 158.1)
- added U8: E32-868T20D, Empreintes:Ebyte, B.Cu at (103.7, 71.0)
- added U9: XC6220B331MR, Package_TO_SOT_SMD:SOT-23-5, F.Cu at (153.9, 154.6)
- J10, J15, J16, J2: value Conn_01x05 -> Conn_01x04; footprint Empreintes:connecteurs5 -> Empreintes:1725672
- J6, J7: footprint Connector_JST:JST_PH_B2B-PH-K_1x02_P2.00mm_Vertical -> Empreintes:SHDR2W90P0X500_1X2_1060X980X1380P
- moved R46 149.4 mm to (174.7, 160.5), turned to 90 degrees
- moved Q7 148.5 mm to (165.3, 156.6)
- moved R31 147.9 mm to (176.1, 160.4), turned to 90 degrees
- moved J20 146.1 mm to (176.6, 152.9), turned to 90 degrees
- moved R45 143.7 mm to (173.3, 160.5), turned to 90 degrees
- moved C55 142.6 mm to (166.6, 150.9), turned to 90 degrees
- moved D10 140.4 mm to (168.6, 155.5), turned to -90 degrees
- moved C56 139.7 mm to (164.9, 151.1), turned to 90 degrees
- moved D11 139.4 mm to (165.6, 154.0), turned to -90 degrees
- moved D12 137.9 mm to (168.8, 152.0), turned to 90 degrees
- moved U1 137.1 mm to (161.7, 148.9), turned to 90 degrees
- moved R41 136.6 mm to (167.0, 148.5)
- moved D14 134.6 mm to (161.4, 155.6)
- moved R49 133.0 mm to (163.1, 154.3)
- moved SW1 132.1 mm to (154.8, 141.8)
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- renumbered C29 to C23, C23 to C24, C30 to C25, C24 to C26, C25 to C27, C31 to C28, C32 to C29, C28 to C30, C34 to C31, C26 to C32, C27 to C34, C43 to C37, C37 to C38, C44 to C39, C38 to C40, C45 to C41, C39 to C42, C46 to C43, C41 to C44, C48 to C45, C40 to C46, C42 to C48, R16 to R12, R17 to R16, R18 to R17, R19 to R18, R20 to R19, R21 to R20, R22 to R21, R23 to R22, R24 to R23, R25 to R24, R26 to R25, R27 to R26, R28 to R27, R29 to R28, R30 to R29, R31 to R30
Connections:
- C15 pad 1: VBAT -> +5V
- C16 pad 1: VBAT -> +5V
- C23 pad 1: Net-(C29-Pad1) -> Net-(C23-Pad1)
- C25 pad 1: Net-(C29-Pad1) -> Net-(C23-Pad1)
- C37 pad 1: Net-(C43-Pad1) -> Net-(C37-Pad1)
- C39 pad 1: Net-(C43-Pad1) -> Net-(C37-Pad1)
- C51 pad 1: VBAT -> +5V
- C52 pad 1: VBAT -> +5V
- IC4 pad 1: SDA -> SD4
- IC4 pad 2: SCL -> SC4
- IC7 pad 11: CLK3 -> CLK4
- IC7 pad 12: DAT3 -> DAT4
- IC8 pad 11: CLK4 -> CLK3
- IC8 pad 12: DAT4 -> DAT3
- J10 pad 1: Net-(C43-Pad1) -> Net-(J10-Pad1)
- J10 pad 2: GND -> Net-(J10-Pad2)
- J10 pad 4: Net-(J10-Pad4) -> Net-(C23-Pad1)
- J15 pad 1: Net-(C22-Pad1) -> Net-(J15-Pad1)
- J15 pad 2: GND -> Net-(J15-Pad2)
- J15 pad 4: Net-(J15-Pad4) -> Net-(C36-Pad1)
- J16 pad 1: Net-(C29-Pad1) -> Net-(J16-Pad1)
- J16 pad 2: GND -> Net-(J16-Pad2)
- J16 pad 4: Net-(J16-Pad4) -> Net-(C37-Pad1)
- J2 pad 1: Net-(C36-Pad1) -> Net-(J2-Pad1)
- J2 pad 2: GND -> Net-(J2-Pad2)
- J2 pad 4: Net-(J2-Pad4) -> Net-(C22-Pad1)
- J6 pad 2: VBAT -> GND
- J7 pad 2: VBAT -> GND
- L3 pad 1: Net-(C29-Pad1) -> Net-(C23-Pad1)
- L5 pad 1: Net-(C43-Pad1) -> Net-(C37-Pad1)
- R17 pad 2: Net-(J15-Pad4) -> Net-(J2-Pad2)
- R18 pad 2: Net-(J15-Pad5) -> Net-(J2-Pad1)
- R21 pad 2: Net-(J16-Pad4) -> Net-(J10-Pad2)
- R22 pad 2: Net-(J16-Pad5) -> Net-(J10-Pad1)
- R25 pad 2: Net-(J2-Pad4) -> Net-(J15-Pad2)
- R26 pad 2: Net-(J2-Pad5) -> Net-(J15-Pad1)
- R29 pad 2: Net-(J10-Pad4) -> Net-(J16-Pad2)
- R30 pad 2: Net-(J10-Pad5) -> Net-(J16-Pad1)
- R7 pad 1: SCL -> SDA
- R8 pad 1: SDA -> SCL
- U3 pad 1: VBAT -> +5V
- U4 pad 13: unconnected-(U4-Pad13) -> SD4
- U4 pad 14: unconnected-(U4-Pad14) -> SC4
- U5 pad 1: VBAT -> +5V
Routing:
- net SD4: track 0.00 -> 78.6 mm, vias 0 -> 2
- net SC4: track 0.00 -> 78.1 mm, vias 0 -> 2
- net EN: track 0.00 -> 71.5 mm, vias 0 -> 2
- net VCC: track 412.2 -> 346.7 mm, vias 13 -> 12
- net +3V3: track 91.4 -> 155.8 mm, vias 3 -> 6
- net UORXD: track 0.00 -> 53.8 mm, vias 0 -> 2
- net UOTXD: track 0.00 -> 53.1 mm, vias 0 -> 2
- net A0/D15: track 52.4 -> 0.00 mm
- net Start_GPS: track 56.3 -> 5.32 mm, vias 2 -> 1
- net VBAT: track 104.4 -> 58.0 mm, vias 3 -> 2
- net DS18b20: track 80.4 -> 44.5 mm
- net RX_GPS: track 58.5 -> 24.6 mm, vias 1 -> 0
- net TX_GPS: track 56.9 -> 23.4 mm, vias 1 -> 0
- net Start_modules: track 33.8 -> 4.56 mm, vias 2 -> 1
- net CLK4: track 27.9 -> 0.00 mm
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Other:
- board size 82.8 x 99.9 mm -> 92.8 x 99.9 mm
- board text removed: "Spare GPIO"

Commit message: update
Parts:
- removed J4: Conn_01x03, Connector_JST:JST_PH_B3B-PH-K_1x03_P2.00mm_Vertical
- removed JP1: SolderJumper_3_Open, Jumper:SolderJumper-3_P1.3mm_Open_RoundedPad1.0x1.5mm_NumberLabels
- removed R42, R43: 1K, Resistor_SMD:R_0603_1608Metric
- added C64: 0.1µF, Capacitor_SMD:C_0603_1608Metric, F.Cu at (141.4, 162.9)
- added IC9: FS312F-G, Empreintes:SOT95P280X145-6N, F.Cu at (141.8, 160.6)
- added Q8: FS8205, Empreintes:FS8205, F.Cu at (141.2, 157.5)
- added R52: 1K, Resistor_SMD:R_0603_1608Metric, F.Cu at (145.8, 160.6)
- added R53: 100, Resistor_SMD:R_0603_1608Metric, F.Cu at (144.5, 162.9)
- moved J19 64.0 mm to (136.9, 94.8)
- moved R7 51.2 mm to (140.6, 129.6)
- moved R8 49.8 mm to (141.4, 127.8)
- moved G*** 10.2 mm to (122.2, 127.1)
- moved G*** 9.56 mm to (131.0, 133.2)
- moved G*** 7.18 mm to (170.4, 163.5)
- moved J13 3.02 mm to (134.5, 78.0)
- moved C19 3.00 mm to (133.2, 88.0)
- moved C5 1.58 mm to (145.8, 149.8), turned to 0 degrees
- moved SW1 0.84 mm to (154.8, 142.7)
- moved J1 0.77 mm to (91.8, 143.0)
- moved D1 0.27 mm to (92.1, 139.3)
- moved R1 0.27 mm to (95.2, 139.3)
- moved R10 0.23 mm to (123.7, 103.2)
- moved J6 0.07 mm to (174.5, 101.6)
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Connections:
- IC7 pad 11: CLK4 -> CLK3
- IC7 pad 12: DAT4 -> DAT3
- IC8 pad 11: CLK3 -> CLK4
- IC8 pad 12: DAT3 -> DAT4
- J19 pad 1: Reset-button -> EN
- U1 pad 13: RXLED -> unconnected-(U1-Pad13)
- U1 pad 14: TXLED -> unconnected-(U1-Pad14)
- U6 pad 1: Net-(U6-Pad1) -> GND
- U6 pad 10: unconnected-(U6-Pad10) -> LORA-TXD-IO
- U6 pad 11: unconnected-(U6-Pad11) -> LORA-RXD-IO
- U6 pad 12: unconnected-(U6-Pad12) -> M1-IO
- U6 pad 17: unconnected-(U6-Pad17) -> TX_GPS
- U6 pad 18: unconnected-(U6-Pad18) -> RX_GPS
- U6 pad 19: unconnected-(U6-Pad19) -> Start_GPS
- U6 pad 22: unconnected-(U6-Pad22) -> INT1
- U6 pad 23: unconnected-(U6-Pad23) -> DS18b20
- U6 pad 27: unconnected-(U6-Pad27) -> IO0
- U6 pad 28: unconnected-(U6-Pad28) -> SD3-CS-D7
- U6 pad 29: unconnected-(U6-Pad29) -> CMD-MOSI-D8
- U6 pad 30: unconnected-(U6-Pad30) -> DAT4
- U6 pad 31: unconnected-(U6-Pad31) -> CLK4
- U6 pad 32: unconnected-(U6-Pad32) -> DAT3
- U6 pad 33: unconnected-(U6-Pad33) -> CLK3
- U6 pad 34: unconnected-(U6-Pad34) -> DAT2
- U6 pad 35: unconnected-(U6-Pad35) -> CLK2
- U6 pad 38: unconnected-(U6-Pad38) -> DAT1
- U6 pad 39: unconnected-(U6-Pad39) -> CLK1
- U6 pad 4: unconnected-(U6-Pad4) -> SDO-MISO-D10
- U6 pad 40: Net-(U6-Pad1) -> GND
- U6 pad 41: Net-(U6-Pad1) -> GND
- U6 pad 5: unconnected-(U6-Pad5) -> CLK-SCK-D9
- U6 pad 8: unconnected-(U6-Pad8) -> LORA-AUX-IO
- U6 pad 9: unconnected-(U6-Pad9) -> M0-IO
- U7 pad 2: GND -> VBAT-
- U8 pad 1: unconnected-(U8-Pad1) -> M0-IO
- U8 pad 2: unconnected-(U8-Pad2) -> M1-IO
- U8 pad 3: unconnected-(U8-Pad3) -> LORA-RXD-IO
- U8 pad 4: unconnected-(U8-Pad4) -> LORA-TXD-IO
- U8 pad 5: unconnected-(U8-Pad5) -> LORA-AUX-IO
- U8 pad 6: unconnected-(U8-Pad6) -> VCC
- U8 pad 7: unconnected-(U8-Pad7) -> GND
Routing:
- net VCC: track 346.7 -> 418.6 mm, vias 12 -> 14
- net VBAT-: track 0.00 -> 61.7 mm, vias 0 -> 2
- net DS18b20: track 44.5 -> 104.5 mm, vias 1 -> 4
- net IO0: track 0.00 -> 36.4 mm
- net M0-IO: track 0.00 -> 35.3 mm, vias 0 -> 2
- net INT1: track 18.9 -> 51.9 mm, vias 1 -> 3
- net CMD-MOSI-D8: track 21.7 -> 50.9 mm
- net SD3-CS-D7: track 22.4 -> 49.9 mm
- net M1-IO: track 0.00 -> 25.5 mm
- net LORA-RXD-IO: track 0.00 -> 22.8 mm
- net DAT4: track 0.00 -> 21.6 mm
- net LORA-TXD-IO: track 0.00 -> 21.3 mm
- net CLK4: track 0.00 -> 21.3 mm
- net LORA-AUX-IO: track 0.00 -> 20.5 mm, vias 0 -> 1
- net RX_GPS: track 24.6 -> 44.4 mm
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Other:
- board text added: "- +"
- board text added: "Solar in"
- board text removed: "- Bat +"
- board text removed: "- Solar in +"
- board text removed: "A0/D15"
- board text removed: "Vcc"

Commit message: update
Routing:
- net GND: vias 287 -> 288
Changed lines of the file:
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@@
   (via (at 92.11 166.6) (size 0.65) (drill 0.3) (layers "F.Cu" "B.Cu") (net 1))
   (via (at 92.6 125.43) (size 0.65) (drill 0.3) (layers "F.Cu" "B.Cu") (free) (net 1))
-  (via (at 143.66 92.65) (size 0.65) (drill 0.3) (layers "F.Cu" "B.Cu") (free) (net 1))
+  (via (at 142.64 96.65) (size 0.65) (drill 0.3) (layers "F.Cu" "B.Cu") (free) (net 1))
   (via (at 130.68875 138.15) (size 0.65) (drill 0.3) (layers "F.Cu" "B.Cu") (free) (net 1))
   (via (at 140.9755 137.13) (size 0.65) (drill 0.3) (layers "F.Cu" "B.Cu") (free) (net 1))
@@
   (via (at 100.1 120.43) (size 0.65) (drill 0.3) (layers "F.Cu" "B.Cu") (free) (net 1))
   (via (at 107.6 117.93) (size 0.65) (drill 0.3) (layers "F.Cu" "B.Cu") (free) (net 1))
+  (via (at 148.85 87.63) (size 0.65) (drill 0.3) (layers "F.Cu" "B.Cu") (free) (net 1))
   (via (at 93.36 167.75) (size 0.65) (drill 0.3) (layers "F.Cu" "B.Cu") (free) (net 1))
   (via (at 97.6 127.93) (size 0.65) (drill 0.3) (layers "F.Cu" "B.Cu") (free) (net 1))
@@
   (segment (start 124.61 96.04) (end 124.61 101.25) (width 0.25) (layer "F.Cu") (net 26))
   (segment (start 88.75 87.03) (end 88.74 87.04) (width 0.25) (layer "F.Cu") (net 26))
-  (segment (start 143.4 102.51) (end 143.605 102.715) (width 0.25) (layer "F.Cu") (net 26))
+  (segment (start 143.605 117.43) (end 143.605 102.746019) (width 0.25) (layer "F.Cu") (net 26))
   (segment (start 103.76 87.03) (end 100.91 87.03) (width 0.25) (layer "F.Cu") (net 26))
   (segment (start 100.91 78.43) (end 100.92 78.43) (width 0.25) (layer "F.Cu") (net 26))
   (segment (start 109.55 86.86) (end 103.77 86.86) (width 0.25) (layer "F.Cu") (net 26))
-  (segment (start 143.605 102.715) (end 143.605 117.43) (width 0.25) (layer "F.Cu") (net 26))
   (segment (start 124.61 101.25) (end 124.64 101.28) (width 0.25) (layer "F.Cu") (net 26))
   (segment (start 109.57 86.84) (end 109.55 86.86) (width 0.25) (layer "F.Cu") (net 26))
   (segment (start 103.79 78.34) (end 103.8 78.35) (width 0.25) (layer "F.Cu") (net 26))
+  (segment (start 143.605 102.746019) (end 143.408481 102.5495) (width 0.25) (layer "F.Cu") (net 26))
   (segment (start 100.91 87.03) (end 100.91 78.43) (width 0.25) (layer "F.Cu") (net 26))
   (segment (start 88.75 78.34) (end 103.79 78.34) (width 0.25) (layer "F.Cu") (net 26))
@@
   (via (at 124.61 96.04) (size 0.65) (drill 0.3) (layers "F.Cu" "B.Cu") (net 26))
   (via (at 124.64 101.28) (size 0.65) (drill 0.3) (layers "F.Cu" "B.Cu") (net 26))
-  (via (at 143.4 102.51) (size 0.65) (drill 0.3) (layers "F.Cu" "B.Cu") (net 26))
+  (via (at 143.408481 102.5495) (size 0.65) (drill 0.3) (layers "F.Cu" "B.Cu") (net 26))
   (segment (start 109.57 86.84) (end 112.19 89.46) (width 0.25) (layer "B.Cu") (net 26))
+  (segment (start 125.909501 102.549501) (end 134.409033 102.549501) (width 0.25) (layer "B.Cu") (net 26))
+  (segment (start 124.64 101.28) (end 125.909501 102.549501) (width 0.25) (layer "B.Cu") (net 26))
   (segment (start 115.95 89.46) (end 119.69 93.2) (width 0.25) (layer "B.Cu") (net 26))
+  (segment (start 143.368981 102.51) (end 143.408481 102.5495) (width 0.25) (layer "B.Cu") (net 26))
   (segment (start 124.42 93.2) (end 124.46 93.16) (width 0.25) (layer "B.Cu") (net 26))
   (segment (start 124.46 93.16) (end 124.61 93.31) (width 0.25) (layer "B.Cu") (net 26))
   (segment (start 119.69 93.2) (end 124.42 93.2) (width 0.25) (layer "B.Cu") (net 26))
-  (segment (start 124.64 101.28) (end 125.9 102.54) (width 0.25) (layer "B.Cu") (net 26))
+  (segment (start 134.448534 102.51) (end 143.368981 102.51) (width 0.25) (layer "B.Cu") (net 26))
+  (segment (start 134.409033 102.549501) (end 134.448534 102.51) (width 0.25) (layer "B.Cu") (net 26))
   (segment (start 124.61 93.31) (end 124.61 96.04) (width 0.25) (layer "B.Cu") (net 26))
   (segment (start 112.19 89.46) (end 115.95 89.46) (width 0.25) (layer "B.Cu") (net 26))
-  (segment (start 125.9 102.54) (end 143.37 102.54) (width 0.25) (layer "B.Cu") (net 26))
-  (segment (start 143.37 102.54) (end 143.4 102.51) (width 0.25) (layer "B.Cu") (net 26))
   (segment (start 110.85875 72.42) (end 109.26125 72.42) (width 0.25) (layer "F.Cu") (net 30))
   (segment (start 135.985 117.43) (end 135.985 127.579296) (width 0.25) (layer "F.Cu") (net 31))
@@
   (segment (start 129.2598 89.9002) (end 131.2898 89.9002) (width 0.25) (layer "B.Cu") (net 51))
   (segment (start 129.26 89.9) (end 128.9445 90.2155) (width 0.25) (layer "B.Cu") (net 51))
-  (segment (start 131.68 103.48) (end 134.13 103.48) (width 0.25) (layer "F.Cu") (net 52))
+  (segment (start 133.508534 103.48) (end 134.819501 102.169033) (width 0.25) (layer "F.Cu") (net 52))
+  (segment (start 134.819501 97.719501) (end 133.59 96.49) (width 0.25) (layer "F.Cu") (net 52))
   (segment (start 133.59 96.49) (end 128.3 96.49) (width 0.25) (layer "F.Cu") (net 52))
-  (segment (start 134.79 102.82) (end 134.79 97.69) (width 0.25) (layer "F.Cu") (net 52))
-  (segment (start 134.13 103.48) (end 134.79 102.82) (width 0.25) (layer "F.Cu") (net 52))
-  (segment (start 134.79 97.69) (end 133.59 96.49) (width 0.25) (layer "F.Cu") (net 52))
+  (segment (start 134.819501 102.169033) (end 134.819501 97.719501) (width 0.25) (layer "F.Cu") (net 52))
+  (segment (start 131.68 103.48) (end 133.508534 103.48) (width 0.25) (layer "F.Cu") (net 52))
   (via (at 128.3 96.49) (size 0.65) (drill 0.3) (layers "F.Cu" "B.Cu") (net 52))
   (segment (start 127.87 89.99) (end 127.87 96.06) (width 0.25) (layer "B.Cu") (net 52))
@@
   (segment (start 154.75 147.66) (end 155.81 147.66) (width 0.25) (layer "F.Cu") (net 113))
   (segment (start 130.065 103.815) (end 130.31 103.57) (width 0.25) (layer "F.Cu") (net 113))
-  (segment (start 132.84 102.21) (end 133.72 101.33) (width 0.25) (layer "F.Cu") (net 113))
   (segment (start 129.39 103.835) (end 129.41 103.815) (width 0.25) (layer "F.Cu") (net 113))
   (segment (start 130.31 102.44) (end 130.54 102.21) (width 0.25) (layer "F.Cu") (net 113))
@@
   (segment (start 156.55 148.4) (end 157.16 148.4) (width 0.25) (layer "F.Cu") (net 113))
   (segment (start 155.81 147.66) (end 156.55 148.4) (width 0.25) (layer "F.Cu") (net 113))
-  (segment (start 131.68 102.21) (end 132.84 102.21) (width 0.25) (layer "F.Cu") (net 113))
   (segment (start 129.41 103.815) (end 130.065 103.815) (width 0.25) (layer "F.Cu") (net 113))
+  (segment (start 131.68 102.21) (end 133.86 102.21) (width 0.25) (layer "F.Cu") (net 113))
+  (segment (start 133.86 102.21) (end 134.17 101.9) (width 0.25) (layer "F.Cu") (net 113))
   (via (at 155.81 147.66) (size 0.65) (drill 0.3) (layers "F.Cu" "B.Cu") (net 113))
-  (via (at 133.72 101.33) (size 0.65) (drill 0.3) (layers "F.Cu" "B.Cu") (net 113))
+  (via (at 134.17 101.9) (size 0.65) (drill 0.3) (layers "F.Cu" "B.Cu") (net 113))
+  (segment (start 136.86 96.56) (end 138.62 98.32) (width 0.25) (layer "B.Cu") (net 113))
+  (segment (start 144.89 102.01) (end 144.78 101.9) (width 0.25) (layer "B.Cu") (net 113))
+  (segment (start 136.86 94.75) (end 136.86 96.56) (width 0.25) (layer "B.Cu") (net 113))
+  (segment (start 144.89 102.07) (end 144.89 102.01) (width 0.25) (layer "B.Cu") (net 113))
+  (segment (start 144.78 101.9) (end 138.56 101.9) (width 0.25) (layer "B.Cu") (net 113))
+  (segment (start 155.81 147.66) (end 145.380489 137.230489) (width 0.25) (layer "B.Cu") (net 113))
   (segment (start 145.380489 137.230489) (end 145.380489 102.560489) (width 0.25) (layer "B.Cu") (net 113))
-  (segment (start 136.86 96.56) (end 138.62 98.32) (width 0.25) (layer "B.Cu") (net 113))
-  (segment (start 138.62 101.33) (end 133.72 101.33) (width 0.25) (layer "B.Cu") (net 113))
-  (segment (start 136.86 94.75) (end 136.86 96.56) (width 0.25) (layer "B.Cu") (net 113))
-  (segment (start 145.380489 102.560489) (end 144.15 101.33) (width 0.25) (layer "B.Cu") (net 113))
-  (segment (start 139.84 101.33) (end 138.62 101.33) (width 0.25) (layer "B.Cu") (net 113))
-  (segment (start 155.81 147.66) (end 145.380489 137.230489) (width 0.25) (layer "B.Cu") (net 113))
-  (segment (start 139.84 101.33) (end 139.78 101.27) (width 0.25) (layer "B.Cu") (net 113))
-  (segment (start 144.15 101.33) (end 139.84 101.33) (width 0.25) (layer "B.Cu") (net 113))
-  (segment (start 138.62 98.32) (end 138.62 101.33) (width 0.25) (layer "B.Cu") (net 113))
+  (segment (start 138.56 101.9) (end 134.17 101.9) (width 0.25) (layer "B.Cu") (net 113))
+  (segment (start 138.62 98.32) (end 138.62 101.84) (width 0.25) (layer "B.Cu") (net 113))
+  (segment (start 145.380489 102.560489) (end 144.89 102.07) (width 0.25) (layer "B.Cu") (net 113))
+  (segment (start 138.62 101.84) (end 138.56 101.9) (width 0.25) (layer "B.Cu") (net 113))
   (segment (start 169.82 150.62) (end 169.85 150.59) (width 0.25) (layer "F.Cu") (net 114))
   (segment (start 171.5075 150.62) (end 169.89 150.62) (width 0.3) (layer "F.Cu") (net 114))

Commit message: update
Parts:
- added AE1: Antenna, Connector_Coaxial:U.FL_Hirose_U.FL-R-SMT-1_Vertical, B.Cu at (128.6, 72.0)
- U8: value E32-868T20D -> RFM95W-868S2; footprint Empreintes:Ebyte -> RF_Module:HOPERF_RFM9XW_SMD
- moved D7 55.1 mm to (129.4, 123.4)
- moved R11 55.1 mm to (132.7, 123.4)
- moved J19 28.3 mm to (143.5, 122.3), turned to -90 degrees
- moved U8 15.7 mm to (117.3, 78.9)
- moved U2 14.1 mm to (141.7, 74.9)
- moved C12 14.1 mm to (151.4, 75.9)
- moved C13 14.1 mm to (146.5, 75.9)
- moved C14 14.1 mm to (144.8, 76.0)
- moved FB1 14.1 mm to (148.9, 76.8)
- moved R13 9.32 mm to (141.2, 93.5)
- moved R14 9.32 mm to (139.7, 93.5)
- moved R15 9.32 mm to (138.1, 93.5)
- moved C19 8.04 mm to (141.2, 87.9)
- moved J13 8.04 mm to (142.5, 77.9)
- moved S1 7.18 mm to (120.3, 90.9)
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Connections:
- U6 pad 15: unconnected-(U6-Pad15) -> Tilt_led_alarm
- U6 pad 20: unconnected-(U6-Pad20) -> LORA-IO12
- U6 pad 21: unconnected-(U6-Pad21) -> LORA-IO13
- U8 pad 1: M0-IO -> GND
- U8 pad 10: unconnected-(U8-Pad10) -> GND
- U8 pad 11: (no net) -> LORA-IO12
- U8 pad 2: M1-IO -> SDO-MISO-D10
- U8 pad 3: LORA-RXD-IO -> CMD-MOSI-D8
- U8 pad 4: LORA-TXD-IO -> CLK-SCK-D9
- U8 pad 5: LORA-AUX-IO -> LORA-NSS-IO
- U8 pad 6: VCC -> LORA-IO3
- U8 pad 7: GND -> LORA-RXD-IO
- U8 pad 8: unconnected-(U8-Pad8) -> GND
- U8 pad 9: unconnected-(U8-Pad9) -> Net-(U8-Pad9)
Routing:
- net LORA-IO12: track 0.00 -> 77.3 mm, vias 0 -> 5
- net LORA-IO13: track 0.00 -> 73.3 mm, vias 0 -> 5
- net M0-IO: track 35.3 -> 85.0 mm, vias 2 -> 3
- net M1-IO: track 25.5 -> 73.0 mm, vias 0 -> 1
- net LORA-RXD-IO: track 22.8 -> 67.3 mm, vias 0 -> 1
- net LORA-TXD-IO: track 21.3 -> 55.4 mm, vias 0 -> 1
- net CMD-MOSI-D8: track 50.9 -> 84.3 mm, vias 2 -> 3
- net CLK-SCK-D9: track 31.1 -> 60.2 mm, vias 2 -> 3
- net SDO-MISO-D10: track 27.2 -> 56.2 mm
- net SCL: track 156.5 -> 139.9 mm
- net SDA: track 160.2 -> 149.0 mm
- net INT1: track 51.9 -> 43.6 mm
- net Tilt_led_alarm: track 1.05 -> 7.05 mm
- net VCC: track 418.6 -> 424.2 mm
- net LORA-AUX-IO: track 20.5 -> 16.9 mm
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
Commit message: update
Parts:
- removed AE1: Antenna, Connector_Coaxial:U.FL_Hirose_U.FL-R-SMT-1_Vertical
- removed U8: RFM95W-868S2, RF_Module:HOPERF_RFM9XW_SMD
- added REF**: Heltec WiFi LoRa V3, Empreintes:Heltec_WiFi_LoRa_V3, F.Cu at (140.2, 118.6)
- J13: moved to F.Cu
- U6: footprint Espressif:ESP32-S3-WROOM-1U -> Espressif:ESP32-S3-WROOM-1
- moved IC4 81.9 mm to (96.4, 70.5), turned to 0 degrees
- moved C10 78.5 mm to (97.8, 72.4), turned to 0 degrees
- moved J13 23.7 mm to (118.9, 77.9), turned to 180 degrees
- moved S1 13.8 mm to (131.8, 83.1)
- moved U6 0.07 mm to (140.4, 107.9)
Connections:
- U6 pad 10: LORA-TXD-IO -> unconnected-(U6-Pad10)
- U6 pad 11: LORA-RXD-IO -> unconnected-(U6-Pad11)
- U6 pad 12: M1-IO -> unconnected-(U6-Pad12)
- U6 pad 14: unconnected-(U6-Pad14) -> Start_modules
- U6 pad 20: LORA-IO12 -> unconnected-(U6-Pad20)
- U6 pad 21: LORA-IO13 -> unconnected-(U6-Pad21)
- U6 pad 8: LORA-AUX-IO -> unconnected-(U6-Pad8)
- U6 pad 9: M0-IO -> unconnected-(U6-Pad9)
Routing:
- net M0-IO: track 85.0 -> 0.00 mm, vias 3 -> 0
- net CMD-MOSI-D8: track 84.3 -> 0.00 mm, vias 3 -> 0
- net LORA-IO12: track 77.3 -> 0.00 mm, vias 5 -> 0
- net LORA-IO13: track 73.3 -> 0.00 mm, vias 5 -> 0
- net M1-IO: track 73.0 -> 0.00 mm, vias 1 -> 0
- net SD4: track 79.0 -> 10.6 mm, vias 2 -> 1
- net SC4: track 78.1 -> 10.4 mm, vias 2 -> 1
- net LORA-RXD-IO: track 67.3 -> 0.00 mm, vias 1 -> 0
- net CLK-SCK-D9: track 60.2 -> 0.00 mm, vias 3 -> 0
- net SDO-MISO-D10: track 56.2 -> 0.00 mm, vias 1 -> 0
- net LORA-TXD-IO: track 55.4 -> 0.00 mm, vias 1 -> 0
- net SD3-CS-D7: track 47.8 -> 0.00 mm, vias 2 -> 0
- net INT1: track 43.6 -> 0.00 mm, vias 3 -> 0
- net VCC: track 424.2 -> 395.4 mm
- net unconnected-(U6-Pad8): track 0.00 -> 16.9 mm, vias 0 -> 1
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Other:
- outline, holes or cut-outs redrawn
