File: ruche.kicad_pcb (KiCad board)
At the start: 2 copper layers, 92.8 x 99.9 mm, 189 parts, among them IC1 CN3791, IC2 MAX17048G+, IC3 L86-M33, IC4 SHT41-AD1B-R3, IC5 HX711, IC6 HX711, IC7 HX711, IC8 HX711, IC9 FS312F-G, J1 Conn_01x02, J10 Conn_01x04, J11 Conn_01x04, J12 Conn_01x04, J13 Micro_SD_Card, J14 Conn_01x03, J15 Conn_01x04, J16 Conn_01x04, J17 Conn_01x04, J18 Conn_01x04, J19 Conn_01x02, J2 Conn_01x04, J20 USB_C_Receptacle_USB2.0 USB41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, J3 Conn_01x03, J5 Conn_01x04, J6 Conn_01x02, J7 Conn_01x02, J8 Conn_01x03, J9 Conn_01x03, Q1 AO3401A, Q2 MMBT4403, Q3 MMBT4403, Q4 MMBT4403, Q5 MMBT4403, Q6 UMH3N, Q7 DMG2301L, Q8 FS8205, SW1 SW_Push, U1 CP2102N-A02-GQFN24, U2 MS5611-01BA, U3 XC6220B331MR, U4 TCA9548APWR, U5 XC6220B331MR, U6 ESP32-S3-WROOM-2, U7 1043, U9 XC6220B331MR

Commit message: update
Parts:
- removed REF**: Heltec WiFi LoRa V3, Empreintes:Heltec_WiFi_LoRa_V3
- added J4: Conn_01x03, Connector_JST:JST_PH_B3B-PH-K_1x03_P2.00mm_Vertical, F.Cu at (163.8, 141.6)
- added JP1: SolderJumper_3_Open, Jumper:SolderJumper-3_P1.3mm_Open_RoundedPad1.0x1.5mm_NumberLabels, B.Cu at (161.0, 144.8)
- U6: footprint Espressif:ESP32-S3-WROOM-1 -> Espressif:ESP32-S3-WROOM-1U
- moved R13 24.5 mm to (116.9, 90.3)
- moved R10 23.7 mm to (141.0, 119.3), turned to 0 degrees
- moved C19 21.9 mm to (119.7, 91.9), turned to -90 degrees
- moved R14 21.6 mm to (118.3, 90.3)
- moved R15 17.4 mm to (121.1, 90.3)
- moved SW1 5.97 mm to (150.8, 138.2), turned to 90 degrees
- moved D7 5.06 mm to (134.4, 124.5), turned to 90 degrees
- moved FID1 4.70 mm to (109.1, 72.3)
- moved R11 2.70 mm to (134.4, 121.3), turned to 90 degrees
- moved U6 0.13 mm to (140.5, 107.9)
Routing:
- net SD3-CS-D7: track 0.00 -> 55.8 mm, vias 0 -> 2
- net CMD-MOSI-D8: track 0.00 -> 53.7 mm, vias 0 -> 2
- net SD4: track 10.6 -> 56.1 mm, vias 1 -> 2
- net SC4: track 10.4 -> 54.6 mm, vias 1 -> 2
- net INT1: track 0.00 -> 42.2 mm, vias 0 -> 1
- net CLK-SCK-D9: track 0.00 -> 34.5 mm, vias 0 -> 2
- net SDO-MISO-D10: track 0.00 -> 29.4 mm, vias 0 -> 2
- net Start_modules: track 4.10 -> 27.9 mm, vias 1 -> 2
- net +3V3: track 163.3 -> 148.9 mm, vias 9 -> 8
- net +5V: track 55.2 -> 68.8 mm
- net Net-(J4-Pad2): track 0.00 -> 8.00 mm
- net DS18b20: track 104.4 -> 108.2 mm, vias 4 -> 3
- net Tilt_led_alarm: track 7.05 -> 3.49 mm
- net VCC: track 395.4 -> 398.7 mm, vias 14 -> 13
- net GND: track 44.3 -> 47.2 mm, vias 277 -> 288
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