File: ruche.kicad_sch (KiCad schematic)
At the start: 40 parts, among them IC2 MAX17048G+, IC3 L86-M33, IC4 SHT41-AD1B-R3, J13 Micro_SD_Card, J19 Conn_01x02, U2 MS5611-01BA, U3 XC6220B331MR, U5 XC6220B331MR

Commit message: update
Parts:
- added C60: 10µF, Capacitor_SMD:C_0603_1608Metric, symbol Device:C
- added C61: 0.1µF, Capacitor_SMD:C_0805_2012Metric, symbol Device:C
- added C62: 0.1µF, Capacitor_SMD:C_0603_1608Metric, symbol Device:C
- added C63: 10µF, Capacitor_SMD:C_0805_2012Metric, symbol Device:C
- added U9: XC6220B331MR, Package_TO_SOT_SMD:SOT-23-5, symbol Regulator_Linear:XC6220B331MR
Connections:
- net +3V3: now also C62.1, C63.1, U9.5 (VOUT)
- net +5V: now also C15.1, C16.1, C51.1, C52.1, U3.1 (VIN), U5.1 (VIN), C60.1, C61.1, U9.1 (VIN), U9.3 (CE)
- net GND: now also C60.2, C61.2, C62.2, C63.2, U9.2 (GND)
- net SCL: now also R8.1; no longer IC4.2 (SCL), R7.1
- net SDA: now also R7.1; no longer IC4.1 (SDA), R8.1
- net VBAT: no longer C15.1, C16.1, C51.1, C52.1, U3.1 (VIN), U5.1 (VIN)
- new net SC4: IC4.2 (SCL)
- new net SD4: IC4.1 (SDA)

Commit message: update
Parts:
- added U8: E32-868T20D, Empreintes:Ebyte, symbol E32-xxxT20D:E32-868T20D
Connections:
- net GND: now also U8.7 (GND)
- net Reset-button: no longer J19.1 (Pin_1)
- net VCC: now also U8.6 (VCC)
- new net EN: J19.1 (Pin_1)
- new net LORA-AUX-IO: U8.5 (AUX)
- new net LORA-RXD-IO: U8.3 (RXD)
- new net LORA-TXD-IO: U8.4 (TXD)
- new net M0-IO: U8.1 (M0)
- new net M1-IO: U8.2 (M1)
Other:
- moved on the sheet: C60, C61, C62, C63, FID1, FID2, FID3, FID4, U9

Commit message: update
Parts:
- removed U8: E32-868T20D, Empreintes:Ebyte, symbol E32-xxxT20D:E32-868T20D
- added AE1: Antenna, Connector_Coaxial:U.FL_Hirose_U.FL-R-SMT-1_Vertical, symbol Device:Antenna
- added U8: RFM95W-868S2, RF_Module:HOPERF_RFM9XW_SMD, symbol RF_Module:RFM95W-868S2
Connections:
- net CLK-SCK-D9: now also U8.4 (SCK)
- net CMD-MOSI-D8: now also U8.3 (MOSI)
- net GND: now also U8.1 (GND), U8.10 (GND), U8.8 (GND)
- net LORA-RXD-IO: now also U8.7 (DIO5)
- net LORA-TXD-IO: now also U8.16 (DIO2)
- net M0-IO: now also U8.14 (DIO0)
- net M1-IO: now also U8.15 (DIO1)
- net SDO-MISO-D10: now also U8.2 (MISO)
- net VCC: now also U8.13 (3.3V)
- new net: AE1.1 (A), U8.9 (ANT)
- new net LORA-IO12: U8.11 (DIO3)
- new net LORA-IO13: U8.12 (DIO4)
- new net LORA-IO3: U8.6 (RESET)
- new net LORA-NSS-IO: U8.5 (NSS)
Other:
- moved on the sheet: FID1, FID3, FID4

Commit message: update
Parts:
- removed AE1: Antenna, Connector_Coaxial:U.FL_Hirose_U.FL-R-SMT-1_Vertical, symbol Device:Antenna
- removed U8: RFM95W-868S2, RF_Module:HOPERF_RFM9XW_SMD, symbol RF_Module:RFM95W-868S2
Other:
- moved on the sheet: FID1, FID2, FID3, FID4
