File: ruched.kicad_sch (KiCad schematic)
At the start: 29 parts

Commit message: update
Parts:
- removed D13: (no value), symbol Device:D_Schottky
- removed JP2: (no value), symbol Jumper:SolderJumper_2_Open
- added U8: E32-868T20D, Empreintes:Ebyte, symbol E32-xxxT20D:E32-868T20D
- C55: value (none) -> 4.7µF; footprint (none) -> Capacitor_SMD:C_0805_2012Metric
- C56, C58: value (none) -> 0.1µF; footprint (none) -> Capacitor_SMD:C_0603_1608Metric
- C57, C59: value (none) -> 22µF; footprint (none) -> Capacitor_SMD:C_0805_2012Metric
- D10, D11, D12: value (none) -> SP1003-01DTG; footprint (none) -> Empreintes:SODFL1406X65N
- D14: value (none) -> D_Schottky; footprint (none) -> Diode_SMD:D_SOD-323
- D8, D9: value (none) -> LED; footprint (none) -> LED_SMD:LED_0603_1608Metric_Castellated
- J20: value (none) -> USB_C_Receptacle_USB2.0 USB4105-GF-A; footprint (none) -> Empreintes:TYPE-C-31-M-12
- Q6: value (none) -> UMH3N; footprint (none) -> Package_TO_SOT_SMD:SOT-363_SC-70-6
- Q7: value (none) -> DMG2301L; footprint (none) -> Package_TO_SOT_SMD:SOT-23
- R31: value (none) -> 1M; footprint (none) -> Resistor_SMD:R_0603_1608Metric
- R41: value (none) -> 22.1K; footprint (none) -> Resistor_SMD:R_0603_1608Metric
- R42, R43, R47: value (none) -> 1K; footprint (none) -> Resistor_SMD:R_0603_1608Metric
- R44: value (none) -> 47.5k; footprint (none) -> Resistor_SMD:R_0603_1608Metric
- R45, R46: value (none) -> 5.1K; footprint (none) -> Resistor_SMD:R_0603_1608Metric
- R48, R49: value (none) -> 10K; footprint (none) -> Resistor_SMD:R_0603_1608Metric
- SW1: value (none) -> SW_Push; footprint (none) -> Empreintes:PTS636SL43SMTRLFS
- U1: value (none) -> CP2102N-A02-GQFN24; footprint (none) -> Package_DFN_QFN:QFN-24-1EP_4x4mm_P0.5mm_EP2.6x2.6mm
- U6: value (none) -> ESP32-S3-WROOM-2; footprint (none) -> Espressif:ESP32-S3-WROOM-1U
Connections:
- net IO0: now also U6.27 (GPIO0/BOOT)
- net RX_GPS: now reaches U6.10 (GPIO17/U1TXD/ADC2_CH6)
- net TX_GPS: now reaches U6.11 (GPIO18/U1RXD/ADC2_CH7/CLK_OUT3)
Other:
- note removed: "Optional"

Commit message: update
Parts:
- removed D8, D9: LED, LED_SMD:LED_0603_1608Metric_Castellated, symbol Device:LED
- removed R42, R43: 1K, Resistor_SMD:R_0603_1608Metric, symbol Device:R
- removed U8: E32-868T20D, Empreintes:Ebyte, symbol E32-xxxT20D:E32-868T20D
- U6: footprint Espressif:ESP32-S3-WROOM-1U -> Espressif:ESP32-S3-WROOM-1; symbol Espressif:ESP32-S3-WROOM-2 -> Espressif:ESP32-S3-WROOM-1
Connections:
- net CLK-SCK-D9: now also U6.5 (GPIO5/TOUCH5/ADC1_CH4)
- net CMD-MOSI-D8: now also U6.29 (SPIIO7/GPIO36/FSPICLK/SUBSPICLK)
- net GND: now also U6.1 (GND), U6.40 (GND), U6.41 (GND)
- net RX_GPS: now also U6.18 (GPIO10/TOUCH10/ADC1_CH9/FSPICS0/FSPIIO4/SUBSPICS0); no longer U6.10 (GPIO17/U1TXD/ADC2_CH6)
- net SD3-CS-D7: now also U6.28 (SPIIO6/GPIO35/FSPID/SUBSPID)
- net SDO-MISO-D10: now also U6.4 (GPIO4/TOUCH4/ADC1_CH3)
- net TX_GPS: now also U6.17 (GPIO9/TOUCH9/ADC1_CH8/FSPIHD/SUBSPIHD); no longer U6.11 (GPIO18/U1RXD/ADC2_CH7/CLK_OUT3)
- net M1-IO: now reaches U6.12 (GPIO8/TOUCH8/ADC1_CH7/SUBSPICS1)
- net Start_GPS: now reaches U6.19 (GPIO11/TOUCH11/ADC2_CH0/FSPID/FSPIIO5/SUBSPID)
- net INT1: now reaches U6.22 (GPIO14/TOUCH14/ADC2_CH3/FSPIWP/FSPIDQS/SUBSPIWP)
- net DS18b20: now reaches U6.23 (GPIO21)
- net DAT4: now reaches U6.30 (SPIDQS/GPIO37/FSPIQ/SUBSPIQ)
- net CLK4: now reaches U6.31 (GPIO38/FSPIWP/SUBSPIWP)
- net DAT3: now reaches U6.32 (MTCK/GPIO39/CLK_OUT3/SUBSPICS1)
- net CLK3: now reaches U6.33 (MTDO/GPIO40/CLK_OUT2)
- net DAT2: now reaches U6.34 (MTDI/GPIO41/CLK_OUT1)
- net CLK2: now reaches U6.35 (MTMS/GPIO42)
- net DAT1: now reaches U6.38 (GPIO2/TOUCH2/ADC1_CH1)
- net CLK1: now reaches U6.39 (GPIO1/TOUCH1/ADC1_CH0)
- net LORA-AUX-IO: now reaches U6.8 (GPIO15/U0RTS/ADC2_CH4/XTAL_32K_P)
- net M0-IO: now reaches U6.9 (GPIO16/U0CTS/ADC2_CH5/XTAL_32K_NH5)
- net RXLED: no longer names the net of U1.13 (GPIO.1)
- net TXLED: no longer names the net of U1.14 (GPIO.0)
- new net LORA-RXD-IO: U6.11 (GPIO18/U1RXD/ADC2_CH7/CLK_OUT3)
- new net LORA-TXD-IO: U6.10 (GPIO17/U1TXD/ADC2_CH6)

Commit message: update
Connections:
- net Tilt_led_alarm: now reaches U6.15 (GPIO3/TOUCH3/ADC1_CH2)
- net LORA-IO12: now reaches U6.20 (GPIO12/TOUCH12/ADC2_CH1/FSPICLK/FSPIIO6/SUBSPICLK)
- net LORA-IO13: now reaches U6.21 (GPIO13/TOUCH13/ADC2_CH2/FSPIQ/FSPIIO7/SUBSPIQ)
Changed lines of the file:
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@@
+    (stroke (width 0) (type default) (color 0 0 0 0))
+  )
+  (wire (pts (xy 140.97 60.96) (xy 147.32 60.96))
     (stroke (width 0) (type default) (color 0 0 0 0))
   )
@@
     (stroke (width 0) (type default) (color 0 0 0 0))
   )
+  (wire (pts (xy 140.97 63.5) (xy 147.32 63.5))
+    (stroke (width 0) (type default) (color 0 0 0 0))
+  )
+  (wire (pts (xy 140.97 38.1) (xy 147.32 38.1))
+    (stroke (width 0) (type default) (color 0 0 0 0))
+  )
   (wire (pts (xy 140.97 43.18) (xy 147.32 43.18))
     (stroke (width 0) (type default) (color 0 0 0 0))
@@
     )
   )
+  (global_label "LORA-IO13" (shape input) (at 140.97 63.5 180) (fields_autoplaced)
+    (effects (font (size 1.27 1.27)) (justify right))
+    (property "Intersheet References" "${INTERSHEET_REFS}" (id 0) (at 128.002 63.4206 0)
+      (effects (font (size 1.27 1.27)) (justify right) hide)
+    )
+  )
+  (global_label "Tilt_led_alarm" (shape output) (at 140.97 38.1 180) (fields_autoplaced)
+    (effects (font (size 1.27 1.27)) (justify right))
+    (property "Intersheet References" "${INTERSHEET_REFS}" (id 0) (at 125.4015 38.0206 0)
+      (effects (font (size 1.27 1.27)) (justify right) hide)
+    )
+  )
   (global_label "CLK4" (shape bidirectional) (at 269.24 66.04 0) (fields_autoplaced)
     (effects (font (size 1.27 1.27)) (justify left))
@@
     )
   )
+  (global_label "LORA-IO12" (shape input) (at 140.97 60.96 180) (fields_autoplaced)
+    (effects (font (size 1.27 1.27)) (justify right))
+    (property "Intersheet References" "${INTERSHEET_REFS}" (id 0) (at 128.002 60.8806 0)
+      (effects (font (size 1.27 1.27)) (justify right) hide)
+    )
+  )
   (global_label "UOTXD" (shape output) (at 267.97 35.56 0) (fields_autoplaced)
     (effects (font (size 1.27 1.27)) (justify left))
@@
     )
   )
+  (global_label "LORA-IO3" (shape input) (at 118.11 35.56 180) (fields_autoplaced)
+    (effects (font (size 1.27 1.27)) (justify right))
+    (property "Intersheet References" "${INTERSHEET_REFS}" (id 0) (at 106.3515 35.4806 0)
+      (effects (font (size 1.27 1.27)) (justify right) hide)
+    )
+  )
   (global_label "DTR" (shape input) (at 78.74 176.53 180) (fields_autoplaced)
     (effects (font (size 1.27 1.27)) (justify right))
@@
     )
   )
+  (global_label "Start_modules" (shape bidirectional) (at 280.67 25.4 180) (fields_autoplaced)
+    (effects (font (size 1.27 1.27)) (justify right))
+    (property "Intersheet References" "${INTERSHEET_REFS}" (id 0) (at 264.8596 25.3206 0)
+      (effects (font (size 1.27 1.27)) (justify right) hide)
+    )
+  )

Commit message: update
Connections:
- net Start_modules: now also U6.14 (GPIO20/U1CTS/ADC2_CH9/CLK_OUT1/USB_D+)
- net LORA-AUX-IO: no longer names the net of U6.8 (GPIO15/U0RTS/ADC2_CH4/XTAL_32K_P)
- net LORA-IO12: no longer names the net of U6.20 (GPIO12/TOUCH12/ADC2_CH1/FSPICLK/FSPIIO6/SUBSPICLK)
- net LORA-IO13: no longer names the net of U6.21 (GPIO13/TOUCH13/ADC2_CH2/FSPIQ/FSPIIO7/SUBSPIQ)
- net LORA-RXD-IO: no longer names the net of U6.11 (GPIO18/U1RXD/ADC2_CH7/CLK_OUT3)
- net LORA-TXD-IO: no longer names the net of U6.10 (GPIO17/U1TXD/ADC2_CH6)
- net M0-IO: no longer names the net of U6.9 (GPIO16/U0CTS/ADC2_CH5/XTAL_32K_NH5)
- net M1-IO: no longer names the net of U6.12 (GPIO8/TOUCH8/ADC1_CH7/SUBSPICS1)
Other:
- moved on the sheet: D10, D12, D14, Q6, R49

Commit message: update
Parts:
- U6: footprint Espressif:ESP32-S3-WROOM-1 -> Espressif:ESP32-S3-WROOM-1U
Changed lines of the file:
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@@
     (property "Reference" "U6" (id 0) (at 201.93 19.1602 0))
     (property "Value" "ESP32-S3-WROOM-2" (id 1) (at 201.93 21.6971 0))
-    (property "Footprint" "Espressif:ESP32-S3-WROOM-1" (id 2) (at 203.2 88.9 0)
+    (property "Footprint" "Espressif:ESP32-S3-WROOM-1U" (id 2) (at 203.2 88.9 0)
       (effects (font (size 1.27 1.27)) hide)
     )
